Commit message: Sim L1: real mount, hemisphere FOV and 5 cm blind zone; stop seeing through walls
The simulated lidar returned no points from a wall 0.25 m ahead and 118 points
from the corridor behind it. Its 0.8 m minimum range is also the GPU near clip,
so anything closer than ~0.46 m was not rendered and rays passed through it.

Now, from docs/L1_LIDAR_REALISM.md:
- Mount from Unitree's radar_joint (under the chin, dome down, 15 deg forward),
  with rays starting 44.5 mm up the dome axis.
- 0..90 deg hemisphere instead of a +-45 deg band, so the sensor no longer sees
  upward directions the real L1 cannot.
- Range 0.05-20 m, noise sigma 1 cm.
- The trunk mesh (which models the dome) and the L1 housing mesh are hidden from
  this lidar only; the legs stay visible as they are to the real sensor.
- 20 Hz render: asking for 15 Hz delivered ~10 Hz in sim time.

Measured standing: wall 0.29 m from the sensor gives 2,269 points on its face
and 0 behind it; 294 returns on the front legs.

The 2D scan band (0.25-1.1 m) no longer matches this sensor; the next commit
replaces it. lidar_check.rviz shows the raw cloud and the scan.

Co-Authored-By: Claude Opus 5.5 <noreply@anthropic.com>

File: unitree_go2_description/urdf/lidar_4D_lidar.xacro (robot description, xacro)
@@ -28,45 +28,90 @@
             </collision>
         </link>
+        <!-- The real mount is radar_joint from Unitree's own go2_description URDF. The
+             link is the L1's mounting face (the SDK frame); its +Z goes through the
+             dome, which here looks down and 15 deg forward from under the chin.
+             See docs/L1_LIDAR_REALISM.md section 5. -->
         <joint name="lidar_l1_joint" type="fixed">
             <parent link="base_link"/>
             <child link="lidar_l1_link"/>
-            <!-- <origin rpy="2.94 0 1.5705" xyz="0.25 -0.038 -0.03"/> -->
-            <origin rpy="2.879 0.0 1.5705" xyz="0.25 -0.038 -0.03"/>
+            <origin rpy="0 2.8782 0" xyz="0.28945 0 -0.046825"/>
         </joint>
-        <gazebo reference="lidar_l1_link">
+        <!-- Ranges are measured from 44.5 mm up the dome axis (SDK z_bias), so the
+             simulated rays start there. -->
+        <link name="lidar_l1_optical"/>
+        <joint name="lidar_l1_optical_joint" type="fixed">
+            <parent link="lidar_l1_link"/>
+            <child link="lidar_l1_optical"/>
+            <origin rpy="0 0 0" xyz="0 0 0.0445"/>
+        </joint>
+        <gazebo reference="lidar_l1_optical">
             <sensor name="lidar_l1" type="gpu_lidar">
                 <topic>unitree_lidar</topic>
-                <update_rate>10</update_rate>
+                <!-- The Go2 publishes /utlidar/cloud at about 15 Hz, but Gazebo
+                     delivered only ~10 Hz when asked for 15, and exactly 20 Hz when
+                     asked for 20 (measured in sim time). Rendering at 20 and thinning
+                     to the real rate is the later point-pattern step. -->
+                <update_rate>20</update_rate>
                 <lidar>
+                    <!-- The L1 sees only the hemisphere on its dome side (0..90 deg
+                         elevation), not a band around its equator. This is a dense
+                         grid over that hemisphere with 1 deg azimuth (max excludes the
+                         duplicate column at +pi) and 1.5 deg elevation (the L1's
+                         pitch step). It is far denser than the real ~1,400 points per
+                         message; matching the real pattern is a later step. -->
                     <scan>
                         <horizontal>
-                            <samples>600</samples>
+                            <samples>360</samples>
                             <resolution>1</resolution>
-                            <min_angle>-3.14159</min_angle>
-                            <max_angle>3.14159</max_angle>
+                            <min_angle>-3.141593</min_angle>
+                            <max_angle>3.124139</max_angle>
                         </horizontal>
                         <vertical>
-                            <samples>30</samples>
+                            <samples>61</samples>
                             <resolution>1</resolution>
-                            <min_angle>-0.785398</min_angle>
-                            <max_angle>0.785398</max_angle>
+                            <min_angle>0</min_angle>
+                            <max_angle>1.570796</max_angle>
                         </vertical>
                     </scan>
+                    <!-- min is also the GPU near clip, so anything closer than ~0.58 x min
+                         is not rendered and the ray returns what lies behind it. At the
+                         old 0.8 m that hid walls up to ~0.46 m away. 0.05 m is the L1's
+                         blind zone. max 20 m is the L1 PM figure until the real unit's
+                         variant is known. -->
                     <range>
-                        <min>0.8</min>
-                        <max>30.0</max>
+                        <min>0.05</min>
+                        <max>20.0</max>
                         <resolution>0.001</resolution>
                     </range>
+                    <!-- Spec accuracy +-2 cm, taken as about 2 sigma. -->
                     <noise>
                         <type>gaussian</type>
                         <mean>0.0</mean>
-                        <stddev>0.008</stddev>
+                        <stddev>0.01</stddev>
                     </noise>
+                    <!-- Ignores visuals flagged 0x2 (see below). -->
+                    <visibility_mask>4294967293</visibility_mask>
                 </lidar>
                 <visualize>false</visualize>
-                <gz_frame_id>lidar_l1_link</gz_frame_id>
+                <gz_frame_id>lidar_l1_optical</gz_frame_id>
                 <always_on>1</always_on>
             </sensor>
         </gazebo>
+        <!-- The rays start inside two solid meshes that on the real robot are the
+             L1's optical window. The trunk mesh models the dome under the chin, and
+             the housing mesh has its origin at a corner, so it wraps the sensor too.
+             Both are hidden from this lidar only. The trunk lies above and behind
+             the downward hemisphere, so little real self-occlusion is lost, and the
+             legs stay visible as they are to the real sensor. -->
+        <gazebo reference="trunk">
+            <visual>
+                <visibility_flags>2</visibility_flags>
+            </visual>
+        </gazebo>
+        <gazebo reference="lidar_l1_link">
+            <visual>
+                <visibility_flags>2</visibility_flags>
+            </visual>
+        </gazebo>
     </xacro:macro>
 </robot>

Commit message: Sim L1: centre the housing mesh on its link
The L1 mesh's origin is a corner of its 75 x 75 mm base, so with the real
(centred) mount the housing was drawn 37 mm to the side and back of the sensor.
The old mount's y = -0.038 had hidden this. Display only; the rays already
started on the centreline.

Co-Authored-By: Claude Opus 5.5 <noreply@anthropic.com>

File: unitree_go2_description/urdf/lidar_4D_lidar.xacro (robot description, xacro)
@@ -2,5 +2,7 @@
 <robot xmlns:xacro="http://www.ros.org/wiki/xacro">
     <xacro:macro name="lidar_l1">
-        <!-- Lidar L1-->
+        <!-- Lidar L1. The mesh's origin is a corner of its 75 x 75 mm base, so it is
+             shifted by half that to put the base centre on the link origin, which is
+             where the SDK frame sits. -->
         <link name="lidar_l1_link">
             <inertial>
@@ -10,5 +12,5 @@
             </inertial>
             <visual>
-                <origin rpy="0 0 0" xyz="0 0 0"/>
+                <origin rpy="0 0 0" xyz="-0.0375 -0.0375 0"/>
                 <geometry>
                     <mesh filename="file://$(find unitree_go2_description)/meshes/L1_4D_Lidar.dae" scale="1 1 1"/>
@@ -19,5 +21,5 @@
             </visual>
             <collision>
-                <origin rpy="0 0 0" xyz="0 0 0"/>
+                <origin rpy="0 0 0" xyz="-0.0375 -0.0375 0"/>
                 <geometry>
                     <mesh filename="file://$(find unitree_go2_description)/meshes/L1_4D_Lidar.dae" scale="1 1 1"/>
